File: eagle/Matrix Clock.brd (EAGLE design)
At the start: 153 x 38 mm, 22 parts, among them IC1 LM1117MPX-3.3, IC4 MAX7219CWG, IC5 MAX7219CWG, IC6 MAX7219CWG, IC7 MAX7219CWG

Commit message: .
Parts:
- added U2: DS3231SN, DS3231SN:SOIC127P1032X265-16N
- U1: value (none) -> ESP-12e
- moved IC1 18.7 mm to (5.00, 43.0)
Connections:
- new net RX: U1.RXD0
- new net TX: U1.TXD0
- new net VBAT: U2.14
- net +3V3: now also U1.CH_PD, U2.2
- net GND: now also U2.10, U2.11, U2.12, U2.13, U2.5, U2.6, U2.7, U2.8, U2.9
- net RESET: now also U2.4
Changed lines of the file:
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@@
 </element>
 <element name="C8" library="rcl" package="C0805" value="0.1mf" x="81.5" y="49.5"/>
-<element name="IC1" library="lm1117" package="SOT223" value="LM1117MPX-3.3" x="8" y="24.5" rot="R90"/>
+<element name="IC1" library="lm1117" package="SOT223" value="LM1117MPX-3.3" x="5" y="43" rot="R90"/>
 <element name="U$1" library="microusb" package="MICRO-USB" value="MICRO-USB" x="1" y="14.5" rot="R270"/>
-<element name="U1" library="esp8266modules" package="ESP12E-SMD" value="" x="138.5" y="19" rot="R270"/>
+<element name="U1" library="esp8266modules" package="ESP12E-SMD" value="ESP-12e" x="138.5" y="19" rot="R270"/>
+<element name="U2" library="DS3231SN" package="SOIC127P1032X265-16N" value="DS3231SN" x="111.5" y="19.5">
+<attribute name="AVAILABILITY" value="Unavailable" x="111.5" y="19.5" size="1.778" layer="27" display="off"/>
+<attribute name="DESCRIPTION" value=" " x="111.5" y="19.5" size="1.778" layer="27" display="off"/>
+<attribute name="MF" value="Maxim Integrated" x="111.5" y="19.5" size="1.778" layer="27" display="off"/>
+<attribute name="MP" value="DS3231SN" x="111.5" y="19.5" size="1.778" layer="27" display="off"/>
+<attribute name="PACKAGE" value="None" x="111.5" y="19.5" size="1.778" layer="27" display="off"/>
+<attribute name="PRICE" value="3.25 USD" x="111.5" y="19.5" size="1.778" layer="27" display="off"/>
+</element>
 </elements>
 <signals>
@@
 <contactref element="IC1" pad="1"/>
 <contactref element="U1" pad="GND"/>
-<wire x1="130.3" y1="10.9" x2="139.44" y2="50.47" width="0" layer="19" extent="1-1"/>
-<wire x1="131.085" y1="52.9392" x2="130.3" y2="10.9" width="0" layer="19" extent="1-16"/>
+<contactref element="U2" pad="13"/>
+<contactref element="U2" pad="5"/>
+<contactref element="U2" pad="7"/>
+<contactref element="U2" pad="10"/>
+<contactref element="U2" pad="11"/>
+<contactref element="U2" pad="12"/>
+<contactref element="U2" pad="8"/>
+<contactref element="U2" pad="9"/>
+<contactref element="U2" pad="6"/>
+<wire x1="131.085" y1="52.9392" x2="139.44" y2="50.47" width="0" layer="19" extent="1-16"/>
 <wire x1="124.735" y1="52.9392" x2="131.085" y2="52.9392" width="0" layer="19" extent="16-16"/>
 <wire x1="113.305" y1="52.9392" x2="124.735" y2="52.9392" width="0" layer="19" extent="16-16"/>
 <wire x1="106.955" y1="52.9392" x2="113.305" y2="52.9392" width="0" layer="19" extent="16-16"/>
-<wire x1="39.525" y1="51.9392" x2="106.955" y2="52.9392" width="0" layer="19" extent="16-16"/>
+<wire x1="97.99" y1="51.47" x2="106.955" y2="52.9392" width="0" layer="19" extent="1-16"/>
+<wire x1="82.45" y1="49.5" x2="97.99" y2="51.47" width="0" layer="19" extent="1-1"/>
+<wire x1="73.49" y1="43.52" x2="82.45" y2="49.5" width="0" layer="19" extent="1-1"/>
+<wire x1="53.44" y1="51.97" x2="73.49" y2="43.52" width="0" layer="19" extent="1-1"/>
+<wire x1="39.525" y1="51.9392" x2="53.44" y2="51.97" width="0" layer="19" extent="1-16"/>
 <wire x1="33.175" y1="51.9392" x2="39.525" y2="51.9392" width="0" layer="19" extent="16-16"/>
 <wire x1="21.745" y1="52.9392" x2="33.175" y2="51.9392" width="0" layer="19" extent="16-16"/>
 <wire x1="15.395" y1="52.9392" x2="21.745" y2="52.9392" width="0" layer="19" extent="16-16"/>
-<wire x1="11.099" y1="22.189" x2="15.395" y2="52.9392" width="0" layer="19" extent="1-16"/>
-<wire x1="2.7" y1="18.225" x2="11.099" y2="22.189" width="0" layer="19" extent="1-1"/>
+<wire x1="7.99" y1="53.47" x2="15.395" y2="52.9392" width="0" layer="19" extent="1-16"/>
+<wire x1="8.099" y1="40.689" x2="15.395" y2="52.9392" width="0" layer="19" extent="1-16"/>
+<wire x1="2.7" y1="18.225" x2="8.099" y2="40.689" width="0" layer="19" extent="1-1"/>
 <wire x1="5.525" y1="13.2" x2="2.7" y2="18.225" width="0" layer="19" extent="1-1"/>
 <wire x1="2.7" y1="10.775" x2="5.525" y2="13.2" width="0" layer="19" extent="1-1"/>
-<wire x1="73.49" y1="43.52" x2="124.735" y2="52.9392" width="0" layer="19" extent="1-16"/>
-<wire x1="82.45" y1="49.5" x2="73.49" y2="43.52" width="0" layer="19" extent="1-1"/>
-<wire x1="97.99" y1="51.47" x2="82.45" y2="49.5" width="0" layer="19" extent="1-1"/>
-<wire x1="53.44" y1="51.97" x2="73.49" y2="43.52" width="0" layer="19" extent="1-1"/>
-<wire x1="7.99" y1="53.47" x2="11.099" y2="22.189" width="0" layer="19" extent="1-1"/>
+<wire x1="116.199" y1="20.135" x2="2.7" y2="10.775" width="0" layer="19" extent="1-1"/>
+<wire x1="116.199" y1="18.865" x2="116.199" y2="20.135" width="0" layer="19" extent="1-1"/>
+<wire x1="116.199" y1="17.595" x2="116.199" y2="18.865" width="0" layer="19" extent="1-1"/>
+<wire x1="116.199" y1="16.325" x2="116.199" y2="17.595" width="0" layer="19" extent="1-1"/>
+<wire x1="116.199" y1="15.055" x2="116.199" y2="16.325" width="0" layer="19" extent="1-1"/>
+<wire x1="106.801" y1="16.325" x2="116.199" y2="16.325" width="0" layer="19" extent="1-1"/>
+<wire x1="106.801" y1="15.055" x2="106.801" y2="16.325" width="0" layer="19" extent="1-1"/>
+<wire x1="106.801" y1="17.595" x2="106.801" y2="16.325" width="0" layer="19" extent="1-1"/>
+<wire x1="106.801" y1="18.865" x2="106.801" y2="17.595" width="0" layer="19" extent="1-1"/>
+<wire x1="130.3" y1="10.9" x2="139.44" y2="50.47" width="0" layer="19" extent="1-1"/>
 </signal>
 <signal name="N$2" class="1">
@@
 <wire x1="17.935" y1="42.8808" x2="35.715" y2="41.8808" width="0" layer="19" extent="16-16"/>
 <wire x1="5.525" y1="15.8" x2="17.935" y2="42.8808" width="0" layer="19" extent="1-16"/>
-<wire x1="11.099" y1="26.811" x2="5.525" y2="15.8" width="0" layer="19" extent="1-1"/>
-<wire x1="6.09" y1="50.51" x2="11.099" y2="26.811" width="0" layer="19" extent="1-1"/>
+<wire x1="8.099" y1="45.311" x2="5.525" y2="15.8" width="0" layer="19" extent="1-1"/>
+<wire x1="6.09" y1="50.51" x2="8.099" y2="45.311" width="0" layer="19" extent="1-1"/>
 <wire x1="6.09" y1="53.47" x2="6.09" y2="50.51" width="0" layer="19" extent="1-1"/>
 <wire x1="52.02" y1="48.51" x2="35.715" y2="41.8808" width="0" layer="19" extent="1-16"/>
@@
 <contactref element="IC1" pad="TAB"/>
 <contactref element="U1" pad="VCC"/>
+<contactref element="U1" pad="CH_PD"/>
+<contactref element="U2" pad="2"/>
+<wire x1="130.3" y1="27.3" x2="140.3" y2="27.3" width="0" layer="19" extent="1-1"/>
 <wire x1="70.77" y1="49.46" x2="130.3" y2="27.3" width="0" layer="19" extent="1-1"/>
-<wire x1="11.099" y1="24.5" x2="70.77" y2="49.46" width="0" layer="19" extent="1-1"/>
-<wire x1="4.901" y1="24.5" x2="11.099" y2="24.5" width="0" layer="19" extent="1-1"/>
+<wire x1="8.099" y1="43" x2="70.77" y2="49.46" width="0" layer="19" extent="1-1"/>
+<wire x1="1.901" y1="43" x2="8.099" y2="43" width="0" layer="19" extent="1-1"/>
+<wire x1="106.801" y1="22.675" x2="1.901" y2="43" width="0" layer="19" extent="1-1"/>
 </signal>
 <signal name="RESET">
 <contactref element="U1" pad="RESET"/>
+<contactref element="U2" pad="4"/>
+<wire x1="106.801" y1="20.135" x2="144.3" y2="27.3" width="0" layer="19" extent="1-1"/>
+</signal>
+<signal name="TX">
+<contactref element="U1" pad="TXD0"/>
+</signal>
+<signal name="RX">
+<contactref element="U1" pad="RXD0"/>
+</signal>
+<signal name="VBAT">
+<contactref element="U2" pad="14"/>
 </signal>
 </signals>
